Commit message: Multiple drones with unique topics added

File: install/rs1_robot/share/rs1_robot/urdf/rs1_drone.urdf.xacro (robot description, xacro)
@@ -1,4 +1,4 @@
 <?xml version="1.0" ?>
-<robot name="rs1_drone" xmlns:xacro="http://www.ros.org/wiki/xacro">
+<robot name="sjtu_drone" xmlns:xacro="http://www.ros.org/wiki/xacro">
 <!-- https://answers.ros.org/question/379014/passing-outside-parameters-into-urdf-file-using-xacro/ -->
   <!-- Need argument to get from launch file -->
@@ -10,11 +10,11 @@
   <xacro:property name="mp" value="${xacro.load_yaml(params_path)}"/>
   <xacro:property name="M_PI" value="3.14159265359" />
-  <link name="$(arg drone_namespace)/base_footprint"/>
+  <link name="base_footprint"/>
   <joint name="base_footprint_joint" type="fixed">
     <origin rpy="0 0 0" xyz="0 0 0"/>
-    <parent link="$(arg drone_namespace)/base_footprint"/>
-    <child link="$(arg drone_namespace)/base_link"/>
-  </joint>
-  <link name="$(arg drone_namespace)/base_link">
+    <parent link="base_footprint"/>
+    <child link="base_link"/>
+  </joint>
+  <link name="base_link">
     <inertial>
       <mass value="1.477"/>
@@ -36,58 +36,60 @@
   </link>
   <joint name="sonar_joint" type="fixed">
-    <parent link="$(arg drone_namespace)/base_link" />
-    <child link="$(arg drone_namespace)/sonar_link" />
+    <parent link="base_link" />
+    <child link="sonar_link" />
     <origin rpy="0 ${M_PI/2} 0" xyz="0 0 0"/>
   </joint>
-  <link name="$(arg drone_namespace)/sonar_link"/>
+  <link name="sonar_link"/>
   <!-- Sonar sensor link -->
   <joint name="down_sonar_joint" type="fixed">
-    <parent link="$(arg drone_namespace)/base_link" />
-    <child link="$(arg drone_namespace)/down_sonar_link" />
+    <parent link="base_link" />
+    <child link="down_sonar_link" />
     <origin rpy="0 ${M_PI/2} 0" xyz="0 0 -0.1"/>
   </joint>
-  <link name="$(arg drone_namespace)/down_sonar_link"/>
+  <link name="down_sonar_link"/>
   <!-- 2D Lidar link -->
   <joint name="lidar_joint" type="fixed">
-    <parent link="$(arg drone_namespace)/base_link" />
-    <child link="$(arg drone_namespace)/lidar_link" />
+    <parent link="base_link" />
+    <child link="lidar_link" />
     <origin rpy="0 0 0" xyz="0 0 0.05"/>
   </joint>
-  <link name="$(arg drone_namespace)/lidar_link"/>
+  <link name="lidar_link"/>
   <joint name="front_cam_joint" type="fixed">
-    <parent link="$(arg drone_namespace)/base_link" />
-    <child link="$(arg drone_namespace)/front_cam_link" />
     <origin rpy="0 0 0" xyz="0.2 0 0"/>
-  </joint>
-  <link name="$(arg drone_namespace)/front_cam_link"/>
+    <parent link="base_link" />
+    <child link="front_cam_link" />
+  </joint>
+  <link name="front_cam_link"/>
   <joint name="bottom_cam_joint" type="fixed">
-    <parent link="$(arg drone_namespace)/base_link" />
-    <child link="$(arg drone_namespace)/bottom_cam_link" />
     <origin rpy="0 ${M_PI/2} 0" xyz="0 0 0"/>
-  </joint>
-  <link name="$(arg drone_namespace)/bottom_cam_link"/>
+    <parent link="base_link" />
+    <child link="bottom_cam_link" />
+  </joint>
+  <link name="bottom_cam_link"/>
   <!-- UPDATED ALL PLUGINS FOR GAZEBO6 FORTRESS COMPATIBILITY -->
   <gazebo>
     <!-- Use native Ignition Gazebo plugins for drone control -->
     <plugin name="ignition::gazebo::systems::VelocityControl" filename="libignition-gazebo6-velocity-control-system.so">
-      <link_name>$(arg drone_namespace)/base_link</link_name>
+      <linkName>base_link</linkName>
     </plugin>
-    <!-- Odometry publisher with proper namespace -->
+    <!-- Odometry publisher -->
     <plugin name="ignition::gazebo::systems::OdometryPublisher" filename="libignition-gazebo6-odometry-publisher-system.so">
-      <odom_frame>$(arg drone_namespace)/odom</odom_frame>
-      <robot_base_frame>$(arg drone_namespace)/base_link</robot_base_frame>
-      <publish_frequency>50</publish_frequency>
+      <odom_frame>${mp['namespace']}/odom</odom_frame>
+      <robot_base_frame>${mp['namespace']}/base_link</robot_base_frame>
+      <odom_publish_frequency>50</odom_publish_frequency>
+      <odom_topic>${mp['namespace']}/odom</odom_topic>
     </plugin>
-    <!-- General Sensors plugin -->
-    <plugin filename="libignition-gazebo6-sensors-system.so" name="ignition::gazebo::systems::Sensors"/>
-  </gazebo>
-  <!-- Update all sensor topics to use namespace -->
-  <gazebo reference="$(arg drone_namespace)/base_link">
+    <!-- General Sensors plugin - REQUIRED for all sensors to work -->
+    <plugin filename="libignition-gazebo6-sensors-system.so" name="ignition::gazebo::systems::Sensors">
+    </plugin>
+  </gazebo>
+  <!-- Note: Fortress uses simplified sensor definitions, bridge handles ROS integration -->
+  <!-- IMU -->
+  <gazebo reference="base_link">
     <sensor name="imu_sensor" type="imu">
-      <topic>$(arg drone_namespace)/imu</topic>
-      <ignition_frame_id>$(arg drone_namespace)/base_link</ignition_frame_id>
       <always_on>true</always_on>
       <visualize>false</visualize>
       <update_rate>100</update_rate>
+      <topic>$(arg drone_namespace)/imu</topic>
       <gz_frame_id>base_link</gz_frame_id>
       <imu>
@@ -152,8 +154,8 @@
   <gazebo reference="down_sonar_link">
     <sensor name="down_sonar" type="gpu_ray">
-      <topic>$(arg drone_namespace)/sonar</topic>
       <always_on>true</always_on>
       <update_rate>50</update_rate>
       <visualize>false</visualize>
+      <topic>model/rs1_drone/sonar</topic>
       <gz_frame_id>down_sonar_link</gz_frame_id>
       <ray>
@@ -182,8 +184,8 @@
   <gazebo reference="lidar_link">
     <sensor name="lidar" type="gpu_ray">
-      <topic>$(arg drone_namespace)/lidar</topic>
       <always_on>true</always_on>
       <update_rate>20</update_rate>
       <visualize>true</visualize>
+      <topic>model/rs1_drone/lidar</topic>
       <gz_frame_id>lidar_link</gz_frame_id>
       <ray>
@@ -212,8 +214,8 @@
   <gazebo reference="front_cam_link">
     <sensor name="front_camera" type="camera">
-      <topic>$(arg drone_namespace)/front_camera</topic>
       <always_on>true</always_on>
       <update_rate>60</update_rate>
       <visualize>false</visualize>
+      <topic>model/rs1_drone/front_camera</topic>
       <gz_frame_id>front_cam_link</gz_frame_id>
       <camera>
@@ -239,8 +241,8 @@
   <gazebo reference="bottom_cam_link">
     <sensor name="bottom_camera" type="camera">
-      <topic>$(arg drone_namespace)/bottom_camera</topic>
       <always_on>true</always_on>
       <update_rate>15</update_rate>
       <visualize>false</visualize>
+      <topic>model/rs1_drone/bottom_camera</topic>
       <gz_frame_id>bottom_cam_link</gz_frame_id>
       <camera>
@@ -266,7 +268,7 @@
   <gazebo reference="base_link">
     <sensor name="gps" type="navsat">
-      <topic>$(arg drone_namespace)/gps</topic>
       <always_on>true</always_on>
       <update_rate>10</update_rate>
+      <topic>model/rs1_drone/gps</topic>
       <gz_frame_id>base_link</gz_frame_id>
       <navsat>
@@ -307,8 +309,8 @@
   <gazebo reference="base_link">
     <sensor name="collision_sensor" type="contact">
-      <topic>$(arg drone_namespace)/bumper</topic>
       <always_on>true</always_on>
       <update_rate>100</update_rate>
-      <ignition_frame_id>$(arg drone_namespace)/base_link</ignition_frame_id>
+      <topic>${mp['namespace']}/bumper</topic>
+      <ignition_frame_id>${mp['namespace']}/base_link</ignition_frame_id>
       <contact>
         <collision>sjtu_drone_collision</collision>
