Commit message: Edited bottom camera orientation and FOV

File: urdf/rs1_drone_adaptive.urdf.xacro (robot description, xacro)
@@ -59,5 +59,5 @@
   <link name="front_cam_link"/>
   <joint name="bottom_cam_joint" type="fixed">
-    <origin rpy="0 ${M_PI/2} 0" xyz="0 0 0"/>
+    <origin rpy="0 ${M_PI/4} 0" xyz="0 0 0"/>
     <parent link="base_link" />
     <child link="bottom_cam_link" />
@@ -247,5 +247,5 @@
       <gz_frame_id>bottom_cam_link</gz_frame_id>
       <camera>
-        <horizontal_fov>1.047</horizontal_fov>
+        <horizontal_fov>1.5</horizontal_fov>
         <image>
           <width>640</width>

Commit message: added theta* path planner

File: urdf/rs1_drone_adaptive.urdf.xacro (robot description, xacro)
@@ -49,5 +49,5 @@
     <parent link="base_link" />
     <child link="lidar_link" />
-    <origin rpy="0 0 0" xyz="0 0 0.05"/>
+    <origin rpy="0 0 0" xyz="0 0 0.25"/>
   </joint>
   <link name="lidar_link"/>

Commit message: Edited bottom camera fov to be 45 deg again, something happened

File: urdf/rs1_drone_adaptive.urdf.xacro (robot description, xacro)
@@ -59,5 +59,5 @@
   <link name="front_cam_link"/>
   <joint name="bottom_cam_joint" type="fixed">
-    <origin rpy="0 ${M_PI/2} 0" xyz="0 0 0"/>
+    <origin rpy="0 ${M_PI/4} 0" xyz="0 0 0"/>
     <parent link="base_link" />
     <child link="bottom_cam_link" />
